File: Hardware/lightning trigger Rev 2/lightning trigger.sch (KiCad schematic (older format))
At the start: 63 parts, among them J1 PJ-237-6A, J2 Conn_02x03_Odd_Even, J3 Conn_01x04, J4 PJ-237-6A, J5 PJ-237-6A, J6 USB_OTG, J7 Conn_01x01, J8 Conn_01x01, J9 PJ-237-6A, Q1 Q_Photo_NPN, Q2 MMBT3904, Q3 BSS138, SW1 SW_SPDT, U1 MCP6001, U10 MCP4532, U11 TLV70233_SOT23-5, U12 TPS2115ADRBR, U2 MCP4532, U3 ATMEGA328P-AU, U4 HM-11, U5 TLP291-4, U6 FS8205, U7 FS312F-G, U8 TP4056, U9 TLP291-4, Y1 Crystal

Commit message: Finished revision 2 of board layout
Parts:
- removed J1, J4, J5, J9: PJ-237-6A, PJ-237-6A:PJ-237-6A, symbol pj-237-6a:PJ-237-6A
- removed J7, J8: Conn_01x01, Pin_Headers:Pin_Header_Straight_1x01_Pitch2.54mm, symbol conn:Conn_01x01
- removed Q3: BSS138, Package_TO_SOT_SMD:SOT-23, symbol Transistor_FET:BSS138
- removed R16, R21, R22: 10k, Resistor_SMD:R_0603_1608Metric, symbol Device:R
- removed R17: 470, Resistor_SMD:R_0603_1608Metric, symbol Device:R
- removed U10, U2: MCP4532, SOP:8-MSOP, symbol lightning-trigger-rescue:MCP4532-Digital_Pots
- removed U12: TPS2115ADRBR, Package_SON:SON-8-1EP_3x2mm_P0.5mm_EP1.4x1.6mm, symbol texas2:TPS2115ADRBR
- removed U6: FS8205, TO_SOT_Packages_SMD:SOT-23-6, symbol fs8205:FS8205
- removed U7: FS312F-G, TO_SOT_Packages_SMD:SOT-23-6, symbol fs312f-g:FS312F-G
- added D2, D3, D4, D5, D6: LED, LED_SMD:LED_0603_1608Metric, symbol Device:LED
- added J3, J4, J5, J6: SJ-2523-SMT, SJ-2523-SMT:SJ-2523-SMT, symbol audio_conn:SJ-2523-SMT
- added J8: Conn_01x02_Female, Connector_JST:JST_PH_S2B-PH-SM4-TB_1x02-1MP_P2.00mm_Horizontal, symbol audio_conn:Conn_01x02_Female
- added J9: Conn_01x02, Resistor_SMD:R_0805_2012Metric, symbol Connector_Generic:Conn_01x02
- added R10, R11, R13, R14, R26, R27, R29, R7, R9: 2k, Resistor_SMD:R_0603_1608Metric, symbol Device:R
- added R4: 150, Resistor_SMD:R_0603_1608Metric, symbol Device:R
- added R5: 10k, Resistor_SMD:R_0603_1608Metric, symbol Device:R
- added U7: AP9211, DFN:U-DFN2030-6, symbol battery_management:AP9211
- C1: Manufacturer P/N C0603C104J5RACTU -> (none); Manufacturer Part Number (none) -> C0603C104J5RACTU
- C10: renamed from C12; Manufacturer P/N C0603C104J5RACTU -> (none); Manufacturer Part Number (none) -> C0603C104J5RACTU
- C11: renamed from C7; Manufacturer P/N C0603C104J5RACTU -> (none); Manufacturer Part Number (none) -> C0603C104J5RACTU
- C12: renamed from C8; Manufacturer P/N C0603C104J5RACTU -> (none); Manufacturer Part Number (none) -> C0603C104J5RACTU
- C2: value 22pF -> 10pF; Manufacturer KEMET -> TDK; Manufacturer P/N C0603C220J1GACTU -> (none); Manufacturer Part Number (none) -> CGA3E2C0G1H100D080AA; Supplier P/N MF-CAP-0603-22pF -> MF-CAP-0603-10pF
- C3: Manufacturer KEMET -> TDK; Manufacturer P/N C0603C220J1GACTU -> (none); Manufacturer Part Number (none) -> CGA3E2C0G1H100D080AA; Supplier P/N MF-CAP-0603-22pF -> MF-CAP-0603-10pF
- C4: renamed from C9; Manufacturer P/N C0603C104J5RACTU -> (none); Manufacturer Part Number (none) -> C0603C104J5RACTU
- C5: renamed from C10; Manufacturer P/N C0603C102J1RACTU -> (none); Manufacturer Part Number (none) -> C0603C102J1RACTU
- C6: renamed from C4; Manufacturer P/N C0603C102J1RACTU -> (none); Manufacturer Part Number (none) -> C0603C102J1RACTU
- C7: renamed from C5; Manufacturer P/N C0603C104J5RACTU -> (none); Manufacturer Part Number (none) -> C0603C104J5RACTU
- C8: renamed from C6; Manufacturer P/N C0603C104J5RACTU -> (none); Manufacturer Part Number (none) -> C0603C104J5RACTU
- C9: renamed from C11; Manufacturer P/N C0603C104J5RACTU -> (none); Manufacturer Part Number (none) -> C0603C104J5RACTU
- D1: Manufacturer P/N DZ2J027M0L -> (none); Manufacturer Part Number (none) -> DZ2J027M0L
- L1: footprint Capacitors_SMD:C_0805 -> Capacitor_SMD:C_0805_2012Metric; Manufacturer (none) -> Bourns; Manufacturer P/N MH2029-300Y -> (none); Manufacturer Part Number (none) -> MH2029-300Y
- MK1: footprint Pin_Headers:Pin_Header_Angled_1x02_Pitch2.54mm -> electret microphone:ELECTRET MICROPHONE; Manufacturer P/N N/A -> (none)
- Q1: Manufacturer P/N SFH 310-2/3 -> (none); Manufacturer Part Number (none) -> SFH 310-2/3
- Q2: Manufacturer P/N MMBT3904LT1G -> (none); Manufacturer Part Number (none) -> MMBT3904LT1G
- R1: renamed from R4; Manufacturer P/N ERJ-3GEYJ103V -> (none); Manufacturer Part Number (none) -> ERJ-3GEYJ103V
- R12: Manufacturer P/N ERJ-3GEYJ202V -> (none); Manufacturer Part Number (none) -> ERJ-3GEYJ202V
- R15: renamed from R8; Manufacturer P/N ERJ-3GEYJ164V -> (none); Manufacturer Part Number (none) -> ERJ-3GEYJ164V
- R16: renamed from R5; Manufacturer P/N ERJ-3GEYJ151V -> (none); Manufacturer Part Number (none) -> ERJ-3GEYJ151V
- R17: renamed from R18; Manufacturer P/N ERJ-3GEYJ151V -> (none); Manufacturer Part Number (none) -> ERJ-3GEYJ151V
- R18: renamed from R6; Manufacturer P/N ERJ-3GEYJ151V -> (none); Manufacturer Part Number (none) -> ERJ-3GEYJ151V
- R19: Manufacturer P/N ERJ-3GEYJ151V -> (none); Manufacturer Part Number (none) -> ERJ-3GEYJ151V
- R2: renamed from R3; Manufacturer P/N ERJ-3GEYJ103V -> (none); Manufacturer Part Number (none) -> ERJ-3GEYJ103V
- R20: renamed from R14; Manufacturer P/N ERJ-3GEYJ202V -> (none); Manufacturer Part Number (none) -> ERJ-3GEYJ202V
- R21: renamed from R7; Manufacturer P/N ERJ-3GEYJ151V -> (none); Manufacturer Part Number (none) -> ERJ-3GEYJ151V
- R22: renamed from R9; Manufacturer P/N ERJ-3GEYJ151V -> (none); Manufacturer Part Number (none) -> ERJ-3GEYJ151V
- R23: renamed from R15; Manufacturer P/N ERJ-3GEYJ151V -> (none); Manufacturer Part Number (none) -> ERJ-3GEYJ151V
- R24: renamed from R10; Manufacturer P/N ERJ-3GEYJ151V -> (none); Manufacturer Part Number (none) -> ERJ-3GEYJ151V
- R25: renamed from R11; Manufacturer P/N ERJ-3GEYJ151V -> (none); Manufacturer Part Number (none) -> ERJ-3GEYJ151V
- R28: renamed from R13; Manufacturer P/N ERJ-3GEYJ202V -> (none); Manufacturer Part Number (none) -> ERJ-3GEYJ202V
- R3: renamed from R1; Manufacturer P/N ERJ-3GEYJ103V -> (none); Manufacturer Part Number (none) -> ERJ-3GEYJ103V
- R6: renamed from R2; Manufacturer P/N ERJ-3GEYJ151V -> (none); Manufacturer Part Number (none) -> ERJ-3GEYJ151V
- R8: renamed from R20; Manufacturer P/N ERJ-3GEYJ470V -> (none); Manufacturer Part Number (none) -> ERJ-3GEYJ470V
- SW1: Manufacturer (none) -> C&K Switches; Manufacturer P/N JS102011SAQN -> (none); Manufacturer Part Number (none) -> JS102011SAQN
- U1: Manufacturer P/N MCP6001T-I/OT -> (none); Manufacturer Part Number (none) -> MCP6001T-I/OT
- U2: renamed from U3; Manufacturer P/N ATMEGA328P-AU -> (none); Manufacturer Part Number (none) -> ATMEGA328P-AU
- U3: renamed from U4; Manufacturer (none) -> Seed; Manufacturer P/N HM-11 -> (none); Manufacturer Part Number (none) -> HM-11
- U4: renamed from U5; Manufacturer (none) -> Toshiba; Manufacturer Part Number (none) -> TLP291-4(GB-TP,E)
- U5: renamed from U11; Manufacturer P/N TLV70233DBVR -> (none); Manufacturer Part Number (none) -> TLV70233DBVR
- U6: renamed from U9; Manufacturer (none) -> Toshiba; Manufacturer Part Number (none) -> TLP291-4(GB-TP,E)
- U8: Manufacturer (none) -> DIOO Microcircuits; Manufacturer P/N TP4056 -> (none); Manufacturer Part Number (none) -> DIO5158; Supplier LCSC -> (none); Supplier P/N C16581 -> (none)
- Y1: footprint Crystals:Crystal_HC18-U_Vertical -> Crystal:Crystal_SMD_2016-4Pin_2.0x1.6mm; Manufacturer (none) -> ECS; Manufacturer P/N N/A -> (none); Manufacturer Part Number (none) -> ECS-160-10-37-JTN-TR
- renumbered J2 to J1, J3 to J2, J6 to J7
Connections:
- net +BATT: now also J8.1 (Pin_1)
- net 3.3V: no longer U3.11 (RST)
- net FOCUS1: now also U4.3; no longer U4.5
- net FOCUS2: now also U4.7; no longer U6.5
- net FOCUS3: now also U6.3; no longer U4.7
- net FOCUS4: now also U2.1 ((PCINT19/OC2B/INT1)PD3)
- net GNDA: now also D1.2 (A), J9.2 (Pin_2), R5.2; no longer C6.2, C8.2
- net GNDD: now also C6.2, C8.2, R12.2, J9.1 (Pin_1), R13.1, R14.1, R29.2, U7.1 (S1), U7.2 (VSS); no longer D1.2 (A)
- net LIGHT_OUT: now also R5.1
- net MICROPHONE_OUT: now also R4.2
- net MISO: now also U6.1; no longer U4.3
- net SHUTTER2: now also U4.5; no longer U6.1
- net SHUTTER4: now also U2.2 ((PCINT20/XCK/T0)PD4), U6.5; no longer U6.3
- net VDD: now also SW1.2 (B), D4.2 (A)
- net VDDA: now also R8.2
- net VUSB: now also R27.2, R7.1
- net at U6.14: now also J5.3; no longer U6.9
- net at U6.13: now also U6.15, J5.1
- net at U6.10: now also J6.3
- net at R6.2, U1.4 (-): now also R4.1
- net at U2.30 ((PCINT16/RXD)PD0): now also U3.2 (TX); no longer U3.4 (RX)
- net at U2.31 ((PCINT17/TXD)PD1): now also R9.2; no longer U3.2 (TX)
- net at U2.32 ((PCINT18/INT0)PD2): now also U3.15 (PIO1), D2.2 (A)
- net at C2.1, U2.7 ((PCINT6/XTAL1/TOSC1)PB6): now also Y1.2; no longer Y1.1
- net at C3.1, U2.8 ((PCINT7/XTAL2/TOSC2)PB7): now also Y1.1; no longer Y1.2
- net at U2.9 ((PCINT21/OC0B/T1)PD5): now also D3.2 (A)
- net at C12.1, R25.1: now also U7.3 (VDD)
- net at U4.14: now also J3.3; no longer U4.9
- net at U4.13: now also U4.15, J3.1
- net at U4.10: now also J4.3
- net at R22.1: now also U6.6; no longer U6.4
- net at R17.1: now also U4.6; no longer U4.4
- net at U4.11: now also U4.9, J4.1; no longer U4.16
- net at U4.12: now also J4.2
- net at R18.1: now also U4.4; no longer U4.6
- net at U6.11: now also U6.9, J6.1; no longer U6.16
- net at U6.12: now also J6.2
- net at R23.1: now also U6.4; no longer U6.6
- net -BAT: no longer names the net of R12.1
- net -BAT: now also R10.2
- net STAT: no longer names the net of U2.19 (ADC6)
- net STAT: now also R11.2, R7.2
- removed net VIN: R8.2, SW1.2 (B)
- net ~CHARGE: no longer names the net of U2.10 ((PCINT22/OC0A/AIN0)PD6)
- net ~CHARGE: no longer U8.7 (~CHRG)
- net ~STDBY: no longer names the net of U2.11 ((PCINT23/AIN1)PD7)
- net ~STDBY: no longer U8.6 (~STDBY)
- new net: D6.1 (K), U8.6 (~STDBY)
- new net: D5.1 (K), U8.7 (~CHRG)
- new net: R10.1, R9.1, U3.4 (RX)
- new net: J3.2, U4.16
- new net: J5.2, U6.16
- new net: D5.2 (A), D6.2 (A), R27.1
- new net: D4.1 (K), R29.1
- new net: D2.1 (K), R13.2
- new net: D3.1 (K), R14.2
- new net: R26.2, U7.5 (VM)
- new net -BATT: J8.2 (Pin_2), R26.1, U7.6 (S2)
Other:
- moved on the sheet: C10, C9, Q1, R20, U3, U4B, U4C, U5, U6B, U6C
